Commit message: add controller manager

File: urdf/first_urdf.urdf.xacro (robot description, xacro)
@@ -68,8 +68,11 @@
       <child link="${wheel_name}"/>
       <dynamics damping="0.7"/>
+      <limit velocity="0.5" effort="1000"/>
     </joint>
     <gazebo reference="${wheel_name}">
-      <mu1>0.2</mu1>
-      <mu2>0.2</mu2>
+      <mu1>200.0</mu1>
+      <mu2>100.0</mu2>
+      <kp value="10000000.0" />
+      <kd value="1.0" />
       <material>Gazebo/Black</material>
     </gazebo>
@@ -77,15 +80,15 @@
       <type>transmission_interface/SimpleTransmission</type>
       <joint name="base_${wheel_name}">
-        <hardwareInterface>hardware_interface/EffortJointInterface</hardwareInterface>
+        <hardwareInterface>hardware_interface/VelocityJointInterface</hardwareInterface>
       </joint>
       <actuator name="${wheel_name}_motor">
-        <hardwareInterface>hardware_interface/EffortJointInterface</hardwareInterface>
+        <hardwareInterface>hardware_interface/VelocityJointInterface</hardwareInterface>
         <mechanicalReducction>1</mechanicalReducction>
       </actuator>
     </transmission>
   </xacro:macro>
-  <xacro:base_wheel_joint wheel_name="lf_wheel" front_end="+1" right_left="+1"/>
-  <xacro:base_wheel_joint wheel_name="lr_wheel" front_end="+1" right_left="-1"/>
-  <xacro:base_wheel_joint wheel_name="bf_wheel" front_end="-1" right_left="+1"/>
+  <xacro:base_wheel_joint wheel_name="fl_wheel" front_end="+1" right_left="+1"/>
+  <xacro:base_wheel_joint wheel_name="fr_wheel" front_end="+1" right_left="-1"/>
+  <xacro:base_wheel_joint wheel_name="bl_wheel" front_end="-1" right_left="+1"/>
   <xacro:base_wheel_joint wheel_name="br_wheel" front_end="-1" right_left="-1"/>
   <!-- world link -->
@@ -102,5 +105,5 @@
   <gazebo>
     <plugin name="gazeo_ros_control" filename="libgazebo_ros_control.so">
-      <robotNamespace>/</robotNamespace>
+      <robotNamespace>/first_urdf</robotNamespace>
       <robotSimType>gazebo_ros_control/DefaultRobotHWSim</robotSimType>
     </plugin>

Commit message: change controllers

File: urdf/first_urdf.urdf.xacro (robot description, xacro)
@@ -36,5 +36,5 @@
   </xacro:macro>
   <!-- link -->
-  <link name="base_link">
+  <link name="car_link">
     <visual>
       <xacro:box_geometry l="${base_length}" w="${base_width}" h="${base_height}"/>
@@ -65,5 +65,5 @@
       <origin xyz="${int(front_end)*base_length*0.3} ${int(right_left)*(base_width*0.5+wheel_length*0.5)} 0.0" rpy="0 0 0"/>
       <axis xyz="0 1 0"/>
-      <parent link="base_link"/>
+      <parent link="car_link"/>
       <child link="${wheel_name}"/>
       <dynamics damping="0.7"/>
@@ -80,8 +80,8 @@
       <type>transmission_interface/SimpleTransmission</type>
       <joint name="base_${wheel_name}">
-        <hardwareInterface>hardware_interface/VelocityJointInterface</hardwareInterface>
+        <hardwareInterface>hardware_interface/EffortJointInterface</hardwareInterface>
       </joint>
       <actuator name="${wheel_name}_motor">
-        <hardwareInterface>hardware_interface/VelocityJointInterface</hardwareInterface>
+        <hardwareInterface>hardware_interface/EffortJointInterface</hardwareInterface>
         <mechanicalReducction>1</mechanicalReducction>
       </actuator>
@@ -93,12 +93,12 @@
   <xacro:base_wheel_joint wheel_name="br_wheel" front_end="-1" right_left="-1"/>
   <!-- world link -->
-  <link name="world"/>
+  <link name="base_link"/>
   <joint name="world_base" type="fixed">
-    <parent link="world"/>
-    <child link="base_link"/>
+    <parent link="base_link"/>
+    <child link="car_link"/>
     <origin xyz="0 0 ${wheel_radius}" rpy="0 0 0"/>
   </joint>
   <!-- material in gazebo -->
-  <gazebo reference="base_link">
+  <gazebo reference="car_link">
     <material>Gazebo/Red</material>
   </gazebo>
@@ -106,5 +106,4 @@
     <plugin name="gazeo_ros_control" filename="libgazebo_ros_control.so">
       <robotNamespace>/first_urdf</robotNamespace>
-      <robotSimType>gazebo_ros_control/DefaultRobotHWSim</robotSimType>
     </plugin>
   </gazebo>

Commit message: change namespace to root

File: urdf/first_urdf.urdf.xacro (robot description, xacro)
@@ -1,4 +1,4 @@
 <?xml version="1.0"?>
-<robot name="myfirst" xmlns:xacro="http://www.ros.org/wiki/xacro">
+<robot name="rbo" xmlns:xacro="http://www.ros.org/wiki/xacro">
   <!-- variables -->
   <xacro:property name="PI" value="3.1415926"/>
@@ -35,6 +35,13 @@
     <origin xyz="${xyz}" rpy="${rpy}"/>
   </xacro:macro>
+  <!-- ros_control plugin -->
+  <gazebo>
+    <plugin name="gazebo_ros_control" filename="libgazebo_ros_control.so">
+      <robotNamespace>/</robotNamespace>
+      <robotSimType>gazebo_ros_control/DefaultRobotHWSim</robotSimType>
+    </plugin>
+  </gazebo>
   <!-- link -->
-  <link name="car_link">
+  <link name="base_link">
     <visual>
       <xacro:box_geometry l="${base_length}" w="${base_width}" h="${base_height}"/>
@@ -65,5 +72,5 @@
       <origin xyz="${int(front_end)*base_length*0.3} ${int(right_left)*(base_width*0.5+wheel_length*0.5)} 0.0" rpy="0 0 0"/>
       <axis xyz="0 1 0"/>
-      <parent link="car_link"/>
+      <parent link="base_link"/>
       <child link="${wheel_name}"/>
       <dynamics damping="0.7"/>
@@ -80,8 +87,8 @@
       <type>transmission_interface/SimpleTransmission</type>
       <joint name="base_${wheel_name}">
-        <hardwareInterface>hardware_interface/EffortJointInterface</hardwareInterface>
+        <hardwareInterface>hardware_interface/VelocityJointInterface</hardwareInterface>
       </joint>
       <actuator name="${wheel_name}_motor">
-        <hardwareInterface>hardware_interface/EffortJointInterface</hardwareInterface>
+        <hardwareInterface>hardware_interface/VelocityJointInterface</hardwareInterface>
         <mechanicalReducction>1</mechanicalReducction>
       </actuator>
@@ -93,18 +100,13 @@
   <xacro:base_wheel_joint wheel_name="br_wheel" front_end="-1" right_left="-1"/>
   <!-- world link -->
-  <link name="base_link"/>
+  <!-- <link name="base_link"/>
   <joint name="world_base" type="fixed">
     <parent link="base_link"/>
     <child link="car_link"/>
     <origin xyz="0 0 ${wheel_radius}" rpy="0 0 0"/>
-  </joint>
+  </joint> -->
   <!-- material in gazebo -->
-  <gazebo reference="car_link">
+  <gazebo reference="base_link">
     <material>Gazebo/Red</material>
   </gazebo>
-  <gazebo>
-    <plugin name="gazeo_ros_control" filename="libgazebo_ros_control.so">
-      <robotNamespace>/first_urdf</robotNamespace>
-    </plugin>
-  </gazebo>
 </robot>
